Commit message: dp_description urdf correction

File: dp_catkin_ws/src/dp_description_pkg/urdf/caster.xacro (robot description, xacro)
@@ -29,4 +29,5 @@
 					<mesh filename="${mesh_caster}"/>
 				</geometry>
+				<material name="white" />
 			</visual>
 			<collision>

File: dp_catkin_ws/src/dp_description_pkg/urdf/roboturdf.xacro (robot description, xacro)
@@ -105,8 +105,8 @@
     </xacro:wheel>
     <xacro:caster caster_prefix="right" parent_link="link_chassis">
-        <origin xyz="${0.065-chassisWidth/2} ${1*(-0.05+boxLength/2)} 0.135" rpy="0 0 0" />
+        <origin xyz="${0.065-chassisWidth/2} ${1*(-0.05+boxLength/2)} 0.135" rpy="0 0 ${PI/2}" />
     </xacro:caster>
     <xacro:caster caster_prefix="left" parent_link="link_chassis">
-        <origin xyz="${0.065-chassisWidth/2} ${-1*(-0.05+boxLength/2)} 0.135" rpy="0 0 0" />
+        <origin xyz="${0.065-chassisWidth/2} ${-1*(-0.05+boxLength/2)} 0.135" rpy="0 0 ${PI/2}" />
     </xacro:caster>
  </robot>
